Commit message: edit xacro

File: visualizer/visualize_simulate/xacro/common_params.xacro (robot description, xacro)
@@ -1,13 +1,15 @@
 <?xml version="1.0"?>
-<!--mathematical parameters-->
-<xacro:properties name="PI" value="3.14"/>
-<!--color parameter-->
-<material name="red">
-    <color rgba="1 0 0 1"/>
-</material>
-<material name="green">
-    <color rgba="0 1 0 1"/>
-</material>
-<material name="blue">
-    <color rgba="0 0 1 1"/>
-</material>
+<robot xmlns:xacro="http://ros.org/wiki/xacro">
+    <!--mathematical parameters-->
+    <xacro:property name="PI" value="3.14"/>
+    <!--color parameter-->
+    <material name="red">
+        <color rgba="1 0 0 1"/>
+    </material>
+    <material name="green">
+        <color rgba="0 1 0 1"/>
+    </material>
+    <material name="blue">
+        <color rgba="0 0 1 1"/>
+    </material>
+</robot>

File: visualizer/visualize_simulate/xacro/object_macro.xacro (robot description, xacro)
@@ -1 +1,80 @@
 <?xml version="1.0"?>
+<robot xmlns:xacro="http://ros.org/wiki/xacro">
+    <xacro:macro name="link_macro" params="suffix parent joint width_parent length_parent height_parent width length height mass ixx ixy ixz iyy iyz izz color">
+        <xacro:if value="${joint=='revolute'}">
+            <joint name="${suffix}_joint" type="revolute">
+                <parent link="${parent}_link"/>
+                <child link="${suffix}"/>
+                <origin xyz="0 0 ${height_parent}" rpy="0 0 0"/>
+                <limit lower="-${PI/2}" upper="${PI/2}" effort="1" velocity="1"/>
+                <axis xyz="0 1 0"/>
+                <dynamics damping="0.0"/>
+            </joint>
+        </xacro:if>
+        <xacro:if value="${joint=='continuous'}">
+            <joint name="${suffix}_joint" type="continuous">
+                <parent link="${parent}_link"/>
+                <child link="${suffix}"/>
+                <origin xyz="0 0 ${height_parent}" rpy="0 0 0"/>
+                <limit effort="0" velocity="1"/>
+                <axis xyz="0 1 0"/>
+                <dynamics damping="0.0"/>
+            </joint>
+        </xacro:if>
+        <link name="${suffix}">
+            <visual>
+                <geometry>
+                    <box size="${width} ${length} ${height}"/>
+                </geometry>
+                <origin xyz="0 0 ${height/2}" rpy="0 0 0"/>
+                <material name="${color}"/>
+            </visual>
+            <inertial>
+                <origin xyz="0 0 0" rpy="0 0 0"/>
+                <mass value="${mass}"/>
+                <inertia
+                    ixx="${ixx}" ixy="${ixy}" ixz="${ixz}"
+                    iyy="${iyy}" iyz="${iyz}"
+                    izz="${izz}"/>
+            </inertial>
+            <collision>
+                <geometry>
+                    <box size="${width} ${length} ${height}"/>
+                </geometry>
+                <origin xyz="0 0 ${height/2}" rpy="0 0 0"/>
+            </collision>
+        </link>
+        <gazebo>
+            <material>Gazebo/Red</material>
+        </gazebo>
+        <joint name="${suffix}_fixed" type="fixed">
+            <parent link="${suffix}"/>
+            <child link="${suffix}_link"/>
+        </joint>
+        <link name="${suffix}_link">
+            <visual>
+                <geometry>
+                    <cylinder radius="${width/2}" length="${length}"/>
+                </geometry>
+                <origin xyz="0 0 ${height}" rpy="${PI/2} 0 0"/>
+                <material name="${color}"/>
+            </visual>
+            <collision>
+                <geometry>
+                    <cylinder radius="${width/2}" length="${length}"/>
+                </geometry>
+                <origin xyz="0 0 ${height}" rpy="${PI/2} 0 0"/>
+            </collision>
+            <inertial>
+                <mass value="0"/>
+                <inertia
+                    ixx="0" ixy="0" ixz="0"
+                    iyy="0" iyz="0"
+                    izz="0"/>
+            </inertial>
+        </link>
+        <gazebo>
+            <material>Gazebo/Red</material>
+        </gazebo>
+    </xacro:macro>
+</robot>

File: visualizer/visualize_simulate/xacro/simple_robot1.xacro (robot description, xacro)
@@ -4,4 +4,5 @@
     <xacro:property name="length" value="0.3"/>
     <xacro:property name="height" value="1.0"/>
+    <xacro:property name="dimension" value="0.1 0.3 1.0"/>
     <xacro:property name="PI" value="3.1415"/>
     <link name="base_link"/>
@@ -13,5 +14,5 @@
         <visual>
             <geometry>
-                <box size="${width} ${length} ${height}" rpy="0 0 0"/>
+                <box size="${dimension}" rpy="0 0 0"/>
             </geometry>
             <material name="red">
