Commit message: added dev branch

File: visualizer/visualize_simulate/xacro/2link.urdf (robot description, URDF)
Before this commit: robot gymnast_robot, 8 links, 7 joints
Links:
- link bar_link: mass None -> 0
Joints:
- joint 1st_joint: limit lower=-1.57 upper=1.57 effort=0 velocity=0 -> effort=0 velocity=1; type revolute -> continuous
- joint 2nd_joint: limit lower=-1.57 upper=1.57 effort=0 velocity=0 -> lower=-1.57 upper=1.57 effort=1 velocity=1
- joint 3rd_joint: limit lower=-1.57 upper=1.57 effort=0 velocity=0 -> lower=-1.57 upper=1.57 effort=1 velocity=1

File: visualizer/visualize_simulate/xacro/2link.xacro (robot description, xacro)
@@ -21,26 +21,43 @@
                 <cylinder radius="0.05" length="1.0"/>
             </geometry>
-            <origin xyz="0 0 3.0" rpy="${PI/2} 0 0"/>
+            <origin xyz="0 0 0.05" rpy="${PI/2} 0 0"/>
         </collision>
+        <inertial>
+            <mass value="0"/>
+            <inertia
+                ixx="0" ixy="0" ixz="0" iyy="0" iyz="0" izz="0" />
+            <origin xyz="0 0 0.05" rpy="${PI/2} 0 0"/>
+        </inertial>
     </link>
-    <gazebo>
+    <gazebo reference="bar_link">
         <material>Gazebo/Orange</material>
     </gazebo>
     <xacro:link_macro
         suffix="1st" parent="bar" joint="continuous"
-        width_parent="0" length_parent="0" height_parent="0.05"
-        width="0.1" length="0.3" height="1.0"
-        mass="0.5" ixx="0.01" ixy="0" ixz="0" iyy="0.01" iyz="0" izz="0.01"
+        x_offset="0" y_offset="0" z_offset="0.05"
+        width="0.1" length="0.3" height="1.0" mass="0.5"
+        ixx="0.01" ixy="0" ixz="0"
+        iyy="0.01" iyz="0"
+        izz="0.01"
         color="red" />
     <xacro:link_macro
         suffix="2nd" parent="1st" joint="revolute"
-        width_parent="0" length_parent="0" height_parent="1.0"
-        width="0.1" length="0.3" height="1.0"
-        mass="0.5" ixx="0.01" ixy="0" ixz="0" iyy="0.01" iyz="0" izz="0.01"
-        color="green"/>
+        x_offset="0" y_offset="0" z_offset="1.0"
+        width="0.1" length="0.3" height="1.0" mass="0.5"
+        ixx="0.01" ixy="0" ixz="0"
+        iyy="0.01" iyz="0"
+        izz="0.01"
+        color="green" />
     <xacro:link_macro suffix="3rd" parent="2nd" joint="revolute"
-        width_parent="0" length_parent="0" height_parent="1.0"
-        width="0.1" length="0.3" height="1.0"
-        mass="0.5" ixx="0.01" ixy="0" ixz="0" iyy="0.01" iyz="0" izz="0.01"
-        color="blue"/>
+        x_offset="0" y_offset="0" z_offset="1.0"
+        width="0.1" length="0.3" height="1.0" mass="0.5"
+        ixx="0.01" ixy="0" ixz="0"
+        iyy="0.01" iyz="0"
+        izz="0.01"
+        color="blue" />
+    <gazebo>
+        <plugin name="gazebo_ros_control" filename="libgazebo_ros_control.so">
+            <robotNamespace>/gymnast_robot</robotNamespace>
+        </plugin>
+    </gazebo>
 </robot>

File: visualizer/visualize_simulate/xacro/object_macro.xacro (robot description, xacro)
@@ -1,10 +1,10 @@
 <?xml version="1.0"?>
 <robot xmlns:xacro="http://ros.org/wiki/xacro">
-    <xacro:macro name="link_macro" params="suffix parent joint width_parent length_parent height_parent width length height mass ixx ixy ixz iyy iyz izz color">
+    <xacro:macro name="link_macro" params="suffix parent joint x_offset y_offset z_offset width length height mass ixx ixy ixz iyy iyz izz color">
         <xacro:if value="${joint=='revolute'}">
             <joint name="${suffix}_joint" type="revolute">
                 <parent link="${parent}_link"/>
                 <child link="${suffix}"/>
-                <origin xyz="0 0 ${height_parent}" rpy="0 0 0"/>
+                <origin xyz="${x_offset} ${y_offset} ${z_offset}" rpy="0 0 0"/>
                 <limit lower="-${PI/2}" upper="${PI/2}" effort="1" velocity="1"/>
                 <axis xyz="0 1 0"/>
@@ -16,5 +16,5 @@
                 <parent link="${parent}_link"/>
                 <child link="${suffix}"/>
-                <origin xyz="0 0 ${height_parent}" rpy="0 0 0"/>
+                <origin xyz="${x_offset} ${y_offset} ${z_offset}" rpy="0 0 0"/>
                 <limit effort="0" velocity="1"/>
                 <axis xyz="0 1 0"/>
@@ -45,5 +45,5 @@
             </collision>
         </link>
-        <gazebo>
+        <gazebo reference="${suffix}">
             <material>Gazebo/Red</material>
         </gazebo>
@@ -74,5 +74,5 @@
             </inertial>
         </link>
-        <gazebo>
+        <gazebo reference="${suffix}_link">
             <material>Gazebo/Red</material>
         </gazebo>

Commit message: changed world to base_link

File: visualizer/visualize_simulate/xacro/2link.urdf (robot description, URDF)
Before this commit: robot gymnast_robot, 8 links, 7 joints
Links:
- removed link base_link
- added link world
Joints:
- joint base_joint: parent base_link -> world

File: visualizer/visualize_simulate/xacro/2link.xacro (robot description, xacro)
@@ -3,7 +3,7 @@
     <xacro:include filename="$(find visualize_simulate)/xacro/common_params.xacro"/>
     <xacro:include filename="$(find visualize_simulate)/xacro/object_macro.xacro"/>
-    <link name="world"/>
+    <link name="base_link"/>
     <joint name="base_joint" type="fixed">
-        <parent link="world"/>
+        <parent link="base_link"/>
         <child link="bar_link"/>
         <origin xyz="0 0 3" rpy="0 ${PI} 0"/>

Commit message: gazebo launched

File: visualizer/visualize_simulate/xacro/2link.urdf (robot description, URDF)
Before this commit: robot gymnast_robot, 9 links, 8 joints
Links:
- link bar_link: mass 0 -> 1
Joints:
- joint 1st_joint: origin xyz=0 0 3 rpy=0 0 0 -> xyz=0 0 0 rpy=0 0 0; parent base_link -> bar_link
- joint system_joint: origin xyz=0 0 3 rpy=0 0 0 -> xyz=0 0.5 3 rpy=0 0 0
- joint world_joint: origin xyz=0 0 0 rpy=0 0 0 -> xyz=0 -0.5 0 rpy=0 0 0

File: visualizer/visualize_simulate/xacro/2link.xacro (robot description, xacro)
@@ -7,5 +7,5 @@
         <parent link="world"/>
         <child link="base_link"/>
-        <origin xyz="0 0 0" rpy="0 0 0"/>
+        <origin xyz="0 -0.5 0" rpy="0 0 0"/>
     </joint>
     <link name="base_link">
@@ -14,9 +14,9 @@
                 <box size="0.1 0.1 3"/>
             </geometry>
-            <origin xyz="0 -0.5 1.5" rpy="0 0 0"/>
-            <material name="blue"/>
+            <origin xyz="0 0 1.5" rpy="0 0 0"/>
+            <material name="Blue"/>
         </visual>
         <inertial>
-            <origin xyz="0 -0.5 1.5" rpy="0 0 0"/>
+            <origin xyz="0 0 1.5" rpy="0 0 0"/>
             <mass value="1"/>
             <inertia ixx="0.1" ixy="0" ixz="0" iyy="0.1" iyz="0" izz="0.1"/>
@@ -26,5 +26,5 @@
                 <box size="0.1 0.1 3"/>
             </geometry>
-            <origin xyz="0 -0.5 1.5" rpy="0 0 0"/>
+            <origin xyz="0 0 1.5" rpy="0 0 0"/>
         </collision>
     </link>
@@ -35,5 +35,5 @@
         <parent link="base_link"/>
         <child link="bar_link"/>
-        <origin xyz="0 0 3" rpy="0 0 0"/>
+        <origin xyz="0 0.5 3" rpy="0 0 0"/>
     </joint>
     <link name="bar_link">
@@ -43,5 +43,5 @@
             </geometry>
             <origin xyz="0 0 0" rpy="${PI/2} 0 0"/>
-            <material name="blue"/>
+            <material name="Orange"/>
         </visual>
         <collision>
@@ -64,17 +64,17 @@
         suffix="1st" parent="bar" joint="continuous"
         x_offset="0" y_offset="0" z_offset="0"
-        width="0.1" length="0.3" height="1.0" mass="0.5"
+        width="0.1" length="0.3" height="0.5" mass="0.5"
         ixx="0.01" ixy="0" ixz="0"
         iyy="0.01" iyz="0"
         izz="0.01"
-        color="red"/>
+        color="Red"/>
     <xacro:link_macro
         suffix="2nd" parent="1st" joint="revolute"
         x_offset="0" y_offset="0" z_offset="1.0"
-        width="0.1" length="0.3" height="1.0" mass="0.5"
+        width="0.1" length="0.3" height="0.5" mass="0.5"
         ixx="0.01" ixy="0" ixz="0"
         iyy="0.01" iyz="0"
         izz="0.01"
-        color="green"/>
+        color="Green"/>
     <xacro:link_macro suffix="3rd" parent="2nd" joint="revolute"
         x_offset="0" y_offset="0" z_offset="1.0"
@@ -83,5 +83,5 @@
         iyy="0.01" iyz="0"
         izz="0.01"
-        color="blue"/>
+        color="Blue"/>
     <gazebo>
         <plugin name="gazebo_ros_control" filename="libgazebo_ros_control.so">

File: visualizer/visualize_simulate/xacro/common_params.xacro (robot description, xacro)
@@ -4,12 +4,15 @@
     <xacro:property name="PI" value="3.14"/>
     <!--color parameter-->
-    <material name="red">
-        <color rgba="1 0 0 1"/>
+    <material name="Red">
+        <color rgba="${255/255} ${0/255} ${0/255} ${255/255}"/>
     </material>
-    <material name="green">
-        <color rgba="0 1 0 1"/>
+    <material name="Green">
+        <color rgba="${0/255} ${255/255} ${0/255} ${255/255}"/>
     </material>
-    <material name="blue">
-        <color rgba="0 0 1 1"/>
+    <material name="Blue">
+        <color rgba="${0/255} ${0/255} ${255/255} ${255/255}"/>
+    </material>
+    <material name="Orange">
+        <color rgba="${255/255} ${108/255} ${10/255} ${255/255}"/>
     </material>
 </robot>

File: visualizer/visualize_simulate/xacro/object_macro.xacro (robot description, xacro)
@@ -46,5 +46,5 @@
         </link>
         <gazebo reference="${suffix}">
-            <material>Gazebo/Red</material>
+            <material>Gazebo/${color}</material>
         </gazebo>
         <joint name="${suffix}_fixed" type="fixed">
@@ -67,14 +67,14 @@
             </collision>
             <inertial>
-                <mass value="0"/>
+                <mass value="0.001"/>
                 <origin xyz="0 0 ${height}" rpy="${PI/2} 0 0"/>
                 <inertia
-                    ixx="0" ixy="0" ixz="0"
-                    iyy="0" iyz="0"
-                    izz="0"/>
+                    ixx="0.001" ixy="0" ixz="0"
+                    iyy="0.001" iyz="0"
+                    izz="0.001"/>
             </inertial>
         </link>
         <gazebo reference="${suffix}_link">
-            <material>Gazebo/Red</material>
+            <material>Gazebo/${color}</material>
         </gazebo>
     </xacro:macro>
