Commit message: xacro base_link to world

File: visualizer/visualize_simulate/xacro/2link.xacro (robot description, xacro)
@@ -3,7 +3,7 @@
     <xacro:include filename="$(find visualize_simulate)/xacro/common_params.xacro"/>
     <xacro:include filename="$(find visualize_simulate)/xacro/object_macro.xacro"/>
-    <link name="base_link"/>
+    <link name="world"/>
     <joint name="base_joint" type="fixed">
-        <parent link="base_link"/>
+        <parent link="world"/>
         <child link="bar_link"/>
         <origin xyz="0 0 3" rpy="0 ${PI} 0"/>

Commit message: controller added

File: visualizer/visualize_simulate/xacro/2link.xacro (robot description, xacro)
@@ -71,5 +71,5 @@
     <xacro:link_macro
         suffix="2nd" parent="1st" joint="revolute"
-        x_offset="0" y_offset="0" z_offset="0.5"
+        x_offset="0" y_offset="0" z_offset="0.55"
         width="0.1" length="0.3" height="0.5" mass="0.5"
         ixx="0.01" ixy="0" ixz="0"
@@ -77,6 +77,7 @@
         izz="0.01"
         color="Green"/>
-    <xacro:link_macro suffix="3rd" parent="2nd" joint="revolute"
-        x_offset="0" y_offset="0" z_offset="0.5"
+    <xacro:link_macro
+        suffix="3rd" parent="2nd" joint="revolute"
+        x_offset="0" y_offset="0" z_offset="0.55"
         width="0.1" length="0.3" height="1.0" mass="0.5"
         ixx="0.01" ixy="0" ixz="0"

File: visualizer/visualize_simulate/xacro/object_macro.xacro (robot description, xacro)
@@ -9,6 +9,14 @@
                 <limit lower="-${PI/2}" upper="${PI/2}" effort="1" velocity="1"/>
                 <axis xyz="0 1 0"/>
-                <dynamics damping="0.1"/>
+                <dynamics damping="0.0"/>
             </joint>
+            <transmission name="${suffix}_transmission">
+                <type>transmission_interface/SimpleTransmission</type>
+                <joint name="${suffix}_joint"/>
+                <actuator name="${suffix}_motor">
+                    <hardwareInterface>EffortJointInterface</hardwareInterface>
+                    <mechanicalReduction>1</mechanicalReduction>
+                </actuator>
+            </transmission>
         </xacro:if>
         <xacro:if value="${joint=='continuous'}">
@@ -19,5 +27,5 @@
                 <limit effort="0" velocity="1"/>
                 <axis xyz="0 1 0"/>
-                <dynamics damping="0.1"/>
+                <dynamics damping="0.0"/>
             </joint>
         </xacro:if>
@@ -47,4 +55,5 @@
         <gazebo reference="${suffix}">
             <material>Gazebo/${color}</material>
+            <selfCollide>true</selfCollide>
         </gazebo>
         <joint name="${suffix}_fixed" type="fixed">
@@ -77,4 +86,5 @@
         <gazebo reference="${suffix}_link">
             <material>Gazebo/${color}</material>
+            <selfCollide>true</selfCollide>
         </gazebo>
     </xacro:macro>

Commit message: adopted for new macro

File: visualizer/visualize_simulate/xacro/2link.xacro (robot description, xacro)
@@ -20,5 +20,6 @@
             <origin xyz="0 0 1.5" rpy="0 0 0"/>
             <mass value="1"/>
-            <inertia ixx="0.1" ixy="0" ixz="0" iyy="0.1" iyz="0" izz="0.1"/>
+            <inertia
+                ixx="0.1" ixy="0" ixz="0" iyy="0.1" iyz="0" izz="0.1"/>
         </inertial>
         <collision>
@@ -64,5 +65,6 @@
         suffix="1st" parent="bar" joint="continuous"
         x_offset="0" y_offset="0" z_offset="0"
-        width="0.1" length="0.3" height="0.5" mass="0.5"
+        width="0.1" length="0.3" height="0.5"
+        mass="0.5" com_x="0" com_y="0" com_z="0"
         ixx="0.01" ixy="0" ixz="0"
         iyy="0.01" iyz="0"
@@ -71,6 +73,7 @@
     <xacro:link_macro
         suffix="2nd" parent="1st" joint="revolute"
-        x_offset="0" y_offset="0" z_offset="0.55"
-        width="0.1" length="0.3" height="0.5" mass="0.5"
+        x_offset="0" y_offset="0" z_offset="0.5"
+        width="0.1" length="0.3" height="0.5"
+        mass="0.5" com_x="0" com_y="0" com_z="0"
         ixx="0.01" ixy="0" ixz="0"
         iyy="0.01" iyz="0"
@@ -79,6 +82,7 @@
     <xacro:link_macro
         suffix="3rd" parent="2nd" joint="revolute"
-        x_offset="0" y_offset="0" z_offset="0.55"
-        width="0.1" length="0.3" height="1.0" mass="0.5"
+        x_offset="0" y_offset="0" z_offset="0.5"
+        mass="0.5" com_x="0" com_y="0" com_z="0"
+        width="0.1" length="0.3" height="1.0"
         ixx="0.01" ixy="0" ixz="0"
         iyy="0.01" iyz="0"
