Commit message: added controller for graduation robot

File: visualizer/visualize_simulate/xacro/grad_robot.xacro (robot description, xacro)
@@ -40,5 +40,5 @@
         <visual>
             <geometry>
-                <cylinder radius="0.05" length="1.0"/>
+                <cylinder radius="0.025" length="1.0"/>
             </geometry>
             <origin xyz="0 0 0" rpy="${PI/2} 0 0"/>
@@ -72,5 +72,5 @@
     <xacro:link_macro
         suffix="2nd" parent="1st" joint="revolute"
-        x_offset="0" y_offset="0" z_offset="0.373"
+        x_offset="0" y_offset="0" z_offset="0.323"
         width="0.05" length="0.15" height="0.265"
         mass="0.351" com_x="0" com_y="0" com_z="0.121"

File: visualizer/visualize_simulate/xacro/object_macro.xacro (robot description, xacro)
@@ -26,5 +26,5 @@
                 <parent link="${parent}_link"/>
                 <child link="${suffix}_link"/>
-                <origin xyz="${x_offset} ${y_offset} ${z_offset}" rpy="0 0 0"/>
+                <origin xyz="${x_offset} ${y_offset} ${z_offset}" rpy="${PI} 0 0"/>
                 <limit effort="0" velocity="1"/>
                 <axis xyz="0 1 0"/>

Commit message: change model plugins

File: visualizer/visualize_simulate/xacro/grad_robot.xacro (robot description, xacro)
@@ -64,5 +64,5 @@
         suffix="1st" parent="bar" joint="continuous"
         x_offset="0" y_offset="0" z_offset="0"
-        width="0.05" length="0.15" height="0.323"
+        width="0.05" length="0.05" height="${0.323+0.015}"
         mass="0.710" com_x="0" com_y="0" com_z="0.232"
         ixx="0.01" ixy="0" ixz="0"
@@ -72,6 +72,6 @@
     <xacro:link_macro
         suffix="2nd" parent="1st" joint="revolute"
-        x_offset="0" y_offset="0" z_offset="0.323"
-        width="0.05" length="0.15" height="0.265"
+        x_offset="0" y_offset="0.05" z_offset="${0.323+0.0015}"
+        width="0.05" length="0.05" height="0.265"
         mass="0.351" com_x="0" com_y="0" com_z="0.121"
         ixx="0.01" ixy="0" ixz="0"
@@ -80,4 +80,16 @@
         color="Green"/>
     <gazebo>
+        <plugin name="ft_sensor" filename="libgazebo_ros_ft_sensor.so">
+            <updateRate>100.0</updateRate>
+            <topicName>1st_sensor/raw</topicName>
+            <jointName>1st_joint</jointName>
+            <gaussianNoise>0.0</gaussianNoise>
+        </plugin>
+        <plugin name="ft_sensor" filename="libgazebo_ros_ft_sensor.so">
+            <updateRate>100.0</updateRate>
+            <topicName>2nd_sensor/raw</topicName>
+            <jointName>2nd_joint</jointName>
+            <gaussianNoise>0.0</gaussianNoise>
+        </plugin>
         <plugin name="gazebo_ros_control" filename="libgazebo_ros_control.so">
             <robotNamespace>/gymnast_robot</robotNamespace>

File: visualizer/visualize_simulate/xacro/object_macro.xacro (robot description, xacro)
@@ -7,5 +7,5 @@
                 <child link="${suffix}_link"/>
                 <origin xyz="${x_offset} ${y_offset} ${z_offset}" rpy="0 0 0"/>
-                <limit lower="-${PI/2}" upper="${PI/2}" effort="1" velocity="1"/>
+                <limit lower="-${PI/2}" upper="${PI/2}" effort="1" velocity="100"/>
                 <axis xyz="0 1 0"/>
                 <dynamics damping="0.0"/>
@@ -18,5 +18,5 @@
                     <actuator name="${suffix}_motor">
                         <hardwareInterface>EffortJointInterface</hardwareInterface>
-                        <mechanicalReduction>1</mechanicalReduction>
+                        <mechanismReduction>1</mechanismReduction>
                     </actuator>
                 </transmission>
@@ -31,8 +31,12 @@
                 <child link="${suffix}_link"/>
                 <origin xyz="${x_offset} ${y_offset} ${z_offset}" rpy="${PI} 0 0"/>
-                <limit effort="0" velocity="1"/>
+                <limit effort="0" velocity="100"/>
                 <axis xyz="0 1 0"/>
                 <dynamics damping="0.0"/>
             </joint>
+            <gazebo reference="${suffix}_joint">
+                <provideFeedback>true</provideFeedback>
+                <turnGravityOff>false</turnGravityOff>
+            </gazebo>
         </xacro:if>
         <link name="${suffix}_link">
@@ -63,12 +67,4 @@
             <selfCollide>true</selfCollide>
         </gazebo>
-        <gazebo>
-            <plugin name="ft_sensor" filename="libgazebo_ros_ft_sensor.so">
-                <updateRate>100.0</updateRate>
-                <topicName>${suffix}_sensor/raw</topicName>
-                <jointName>${suffix}_joint</jointName>
-                <gaussianNoise>0.0</gaussianNoise>
-            </plugin>
-        </gazebo>
     </xacro:macro>
 </robot>
