Commit message: change mass & xacro

File: my_robot/urdf/my_robot03.urdf (robot description, URDF)
Before this commit: robot my_robot, 7 links, 6 joints
Links:
- link arm1_link: mass 0.08 -> 1.0
- link arm2_link: mass 0.08 -> 0.001; geometry collision box size=1.2 0.1 0.1; visual box size=1.2 0.1 0.1
- link arm3_link: mass 3 -> 1.0
- link base_link: mass 1 -> 10
- link guide1_link: geometry collision box size=0.7 0.1 0.1; visual box size=0.7 0.1 0.1
Joints:
- joint arm1_joint: limit lower=-0.5 upper=1.5 effort=40 velocity=10 -> (none); origin xyz=-0.7071 0.1 0.7071 rpy=0 0 0 -> xyz=0 0.1 1.2071 rpy=0 0 0; type revolute -> continuous
- joint arm2_joint: origin xyz=0 0 0.6 rpy=0 0 0 -> xyz=0 0 1 rpy=0 0 0
- joint guide1_joint: limit lower=-1.0 upper=3.0 effort=1000 velocity=100 -> lower=0.0 upper=4.0 effort=1000 velocity=100; origin xyz=0.6 -0.1 1.5 rpy=0 ${-1*pi/2} 0 -> xyz=1.5 -0.1 0.8071 rpy=0 -1.5708 0

File: visualizer/visualize_simulate/xacro/2link.urdf (robot description, URDF)
Before this commit: robot gymnast_robot, 8 links, 7 joints
Links:
- added link base_link, mass 1; collision box size=0.1 0.1 3; visual box size=0.1 0.1 3
Joints:
- removed joint base_joint
- added joint system_joint: type fixed, parent base_link, child bar_link, origin xyz=0 0 3 rpy=0 0 0
- added joint world_joint: type fixed, parent world, child base_link, origin xyz=0 0 0 rpy=0 0 0
- joint 1st_joint: origin xyz=0 0 0.05 rpy=0 0 0 -> xyz=0 0 3 rpy=0 0 0; parent bar_link -> base_link

File: visualizer/visualize_simulate/xacro/2link.xacro (robot description, xacro)
@@ -3,9 +3,37 @@
     <xacro:include filename="$(find visualize_simulate)/xacro/common_params.xacro"/>
     <xacro:include filename="$(find visualize_simulate)/xacro/object_macro.xacro"/>
-    <link name="base_link"/>
-    <joint name="base_joint" type="fixed">
+    <link name="world"/>
+    <joint name="world_joint" type="fixed">
+        <parent link="world"/>
+        <child link="base_link"/>
+        <origin xyz="0 0 0" rpy="0 0 0"/>
+    </joint>
+    <link name="base_link">
+        <visual>
+            <geometry>
+                <box size="0.1 0.1 3"/>
+            </geometry>
+            <origin xyz="0 -0.5 1.5" rpy="0 0 0"/>
+            <material name="blue"/>
+        </visual>
+        <inertial>
+            <origin xyz="0 -0.5 1.5" rpy="0 0 0"/>
+            <mass value="1"/>
+            <inertia ixx="0.1" ixy="0" ixz="0" iyy="0.1" iyz="0" izz="0.1"/>
+        </inertial>
+        <collision>
+            <geometry>
+                <box size="0.1 0.1 3"/>
+            </geometry>
+            <origin xyz="0 -0.5 1.5" rpy="0 0 0"/>
+        </collision>
+    </link>
+    <gazebo reference="base_link">
+        <material>Gazebo/Blue</material>
+    </gazebo>
+    <joint name="system_joint" type="fixed">
         <parent link="base_link"/>
         <child link="bar_link"/>
-        <origin xyz="0 0 3" rpy="0 ${PI} 0"/>
+        <origin xyz="0 0 3" rpy="0 0 0"/>
     </joint>
     <link name="bar_link">
@@ -14,5 +42,5 @@
                 <cylinder radius="0.05" length="1.0"/>
             </geometry>
-            <origin xyz="0 0 0.05" rpy="${PI/2} 0 0"/>
+            <origin xyz="0 0 0" rpy="${PI/2} 0 0"/>
             <material name="blue"/>
         </visual>
@@ -21,11 +49,11 @@
                 <cylinder radius="0.05" length="1.0"/>
             </geometry>
-            <origin xyz="0 0 0.05" rpy="${PI/2} 0 0"/>
+            <origin xyz="0 0 0" rpy="${PI/2} 0 0"/>
         </collision>
         <inertial>
-            <mass value="0"/>
+            <mass value="1"/>
             <inertia
-                ixx="0" ixy="0" ixz="0" iyy="0" iyz="0" izz="0" />
-            <origin xyz="0 0 0.05" rpy="${PI/2} 0 0"/>
+                ixx="0.1" ixy="0" ixz="0" iyy="0.1" iyz="0" izz="0.1"/>
+            <origin xyz="0 0 0" rpy="${PI/2} 0 0"/>
         </inertial>
     </link>
@@ -35,10 +63,10 @@
     <xacro:link_macro
         suffix="1st" parent="bar" joint="continuous"
-        x_offset="0" y_offset="0" z_offset="0.05"
+        x_offset="0" y_offset="0" z_offset="0"
         width="0.1" length="0.3" height="1.0" mass="0.5"
         ixx="0.01" ixy="0" ixz="0"
         iyy="0.01" iyz="0"
         izz="0.01"
-        color="red" />
+        color="red"/>
     <xacro:link_macro
         suffix="2nd" parent="1st" joint="revolute"
@@ -48,5 +76,5 @@
         iyy="0.01" iyz="0"
         izz="0.01"
-        color="green" />
+        color="green"/>
     <xacro:link_macro suffix="3rd" parent="2nd" joint="revolute"
         x_offset="0" y_offset="0" z_offset="1.0"
@@ -55,5 +83,5 @@
         iyy="0.01" iyz="0"
         izz="0.01"
-        color="blue" />
+        color="blue"/>
     <gazebo>
         <plugin name="gazebo_ros_control" filename="libgazebo_ros_control.so">

File: visualizer/visualize_simulate/xacro/object_macro.xacro (robot description, xacro)
@@ -9,5 +9,5 @@
                 <limit lower="-${PI/2}" upper="${PI/2}" effort="1" velocity="1"/>
                 <axis xyz="0 1 0"/>
-                <dynamics damping="0.0"/>
+                <dynamics damping="0.1"/>
             </joint>
         </xacro:if>
@@ -19,5 +19,5 @@
                 <limit effort="0" velocity="1"/>
                 <axis xyz="0 1 0"/>
-                <dynamics damping="0.0"/>
+                <dynamics damping="0.1"/>
             </joint>
         </xacro:if>
@@ -68,4 +68,5 @@
             <inertial>
                 <mass value="0"/>
+                <origin xyz="0 0 ${height}" rpy="${PI/2} 0 0"/>
                 <inertia
                     ixx="0" ixy="0" ixz="0"
