Commit message: reshaped code

File: visualizer/simulate_robot/urdf/acrobat_robot_IB.xacro (robot description, xacro)
@@ -47,3 +47,11 @@
         iyy="0.01" iyz="0"
         izz="0.0058"/>
+    <!-- 2nd_link -->
+    <xacro:link_macro
+        suffix="2nd_link" parent="1st_link" type="revolute" color="green"
+        width="${width2}" length="${length2}" height="${height2}" x_offset="0" y_offset="${width2}" z_offset="${height1}"
+        mass="${mass1}" comx="${comx2}" comy="${comy2}" comz="${comz2}"
+        ixx="0.01" ixy="0" ixz="0"
+        iyy="0.01" iyz="0"
+        izz="0.070"/>
 </robot>

File: visualizer/simulate_robot/urdf/link_macro.xacro (robot description, xacro)
@@ -1,69 +1,69 @@
 <?xml version="1.0"?>
 <robot xmlns:xacro="http://www.ros.org/wiki/xacro">
-    <xacro:macro name="link_macro"
-        params="suffix parent type color
-        width length height x_offset y_offset z_offset
-        mass comx comy comz
-        ixx ixy ixz
-        iyy iyz
-        izz">
-        <!-- revolute joint(actuated) -->
-        <xacro:if value="${type=='revolute'}">
-            <joint name="${suffix}_joint" type="revolute">
-                <parent link="${parent}"/>
-                <child link="${suffix}"/>
-                <origin xyz="${x_offset} ${y_offset} ${z_offset}" rpy="0 0 0"/>
-                <limit upper="${PI/2}" lower="${PI/2}" effort="100" velocity="100"/>
-                <axis xyz="0 1 0"/>
-                <dynamics damping="0.1"/>
-            </joint>
-        </xacro:if>
-        <!-- continuous joint(passive) -->
-        <xacro:if value="${type=='continuous'}">
-            <joint name="${suffix}_joint" type="continuous">
-                <parent link="${parent}"/>
-                <child link="${suffix}"/>
-                <origin xyz="${x_offset} ${y_offset} ${z_offset}" rpy="0 0 0"/>
-                <limit effort="100" velocity="100"/>
-                <axis xyz="0 1 0"/>
-                <dynamics damping="0.00001"/>
-            </joint>
-        </xacro:if>
-        <link name="${suffix}">
-            <!-- visual config -->
-            <visual>
-                <origin xyz="0 0 ${height/2}" rpy="0 0 0"/>
-                <material name="${color}"/>
-                <geometry>
-                    <box size="${width} ${length} ${height}"/>
-                </geometry>
-            </visual>
-            <!-- Gazebo collision config -->
-            <collision>
-                <origin xyz="0 0 ${height/2}" rpy="0 0 0"/>
-                <geometry>
-                    <box size="${width} ${length} ${height}"/>
-                </geometry>
-            </collision>
-            <!-- inertial config -->
-            <inertial>
-                <origin xyz="${comx} ${comy} ${comz}" rpy="0 0 0"/>
-                <mass value="${mass}"/>
-                <inertia
-                    ixx="${ixx}" ixy="${ixy}" ixz="${ixz}"
-                    iyy="${iyy}" iyz="${iyz}"
-                    izz="${izz}"/>
-            </inertial>
-        </link>
-        <transmission name="${suffix}_transmission">
-            <type>transmission_interface/SimpleTransmission</type>
-            <joint name="${suffix}_joint">
-                <hardwareInterface>hardware_interface/EffortJointInterface</hardwareInterface>
-            </joint>
-            <actuator name="${suffix}_motor">
-            <hardwareInterface>hardware_interface/EffortJointInterface</hardwareInterface>
-            <mechanicalReduction>1</mechanicalReduction>
-            </actuator>
-        </transmission>
-    </xacro:macro>
+  <xacro:macro name="link_macro"
+    params="suffix parent type color
+    width length height x_offset y_offset z_offset
+    mass comx comy comz
+    ixx ixy ixz
+    iyy iyz
+    izz">
+    <!-- revolute joint(actuated) -->
+    <xacro:if value="${type=='revolute'}">
+      <joint name="${suffix}_joint" type="revolute">
+        <parent link="${parent}"/>
+        <child link="${suffix}"/>
+        <origin xyz="${x_offset} ${y_offset} ${z_offset}" rpy="0 0 0"/>
+        <limit upper="${PI/2}" lower="${-PI/2}" effort="100" velocity="100"/>
+          <axis xyz="0 1 0"/>
+          <dynamics damping="0.1"/>
+      </joint>
+    </xacro:if>
+    <!-- continuous joint(passive) -->
+    <xacro:if value="${type=='continuous'}">
+        <joint name="${suffix}_joint" type="continuous">
+          <parent link="${parent}"/>
+          <child link="${suffix}"/>
+          <origin xyz="${x_offset} ${y_offset} ${z_offset}" rpy="0 0 0"/>
+          <limit effort="0" velocity="100"/>
+          <axis xyz="0 1 0"/>
+          <dynamics damping="0.00001"/>
+        </joint>
+   </xacro:if>
+    <link name="${suffix}">
+      <!-- visual config -->
+      <visual>
+        <origin xyz="0 0 ${height/2}" rpy="0 0 0"/>
+        <material name="${color}"/>
+          <geometry>
+            <box size="${width} ${length} ${height}"/>
+          </geometry>
+      </visual>
+      <!-- Gazebo collision config -->
+      <collision>
+        <origin xyz="0 0 ${height/2}" rpy="0 0 0"/>
+          <geometry>
+            <box size="${width} ${length} ${height}"/>
+          </geometry>
+      </collision>
+      <!-- inertial config -->
+      <inertial>
+        <origin xyz="${comx} ${comy} ${comz}" rpy="0 0 0"/>
+        <mass value="${mass}"/>
+        <inertia
+          ixx="${ixx}" ixy="${ixy}" ixz="${ixz}"
+          iyy="${iyy}" iyz="${iyz}"
+          izz="${izz}"/>
+      </inertial>
+    </link>
+    <transmission name="${suffix}_transmission">
+      <type>transmission_interface/SimpleTransmission</type>
+      <joint name="${suffix}_joint">
+        <hardwareInterface>hardware_interface/EffortJointInterface</hardwareInterface>
+      </joint>
+      <actuator name="${suffix}_motor">
+        <hardwareInterface>hardware_interface/EffortJointInterface</hardwareInterface>
+        <mechanicalReduction>1</mechanicalReduction>
+      </actuator>
+    </transmission>
+  </xacro:macro>
 </robot>

File: visualizer/simulate_robot/urdf/system_constants.xacro (robot description, xacro)
@@ -1,23 +1,23 @@
 <?xml version="1.0"?>
 <robot xmlns:xacro="http://www.ros.org/wiki/xacro">
-    <!-- Robot constants parameter -->
-    <!-- Y up,X front -->
-    <!-- Link 1 -->
-    <xacro:property name="mass1" value="0.710"/>
-    <xacro:property name="length1" value="0.05"/>
-    <xacro:property name="width1" value="0.05"/>
-    <xacro:property name="height1" value="${0.323+0.015}"/> <!-- length + joint -->
-    <xacro:property name="comx1" value="0.0"/>
-    <xacro:property name="comy1" value="0.0"/>
-    <xacro:property name="comz1" value="0.232"/>
-    <!-- Link 2 -->
-    <xacro:property name="mass2" value="0.351"/>
-    <xacro:property name="length2" value="0.05"/>
-    <xacro:property name="width2" value="0.05"/>
-    <xacro:property name="height2" value="0.265"/>
-    <xacro:property name="comx2" value="0.0"/>
-    <xacro:property name="comy2" value="0.0"/>
-    <xacro:property name="comz2" value="0.265"/>
-    <!-- World constants parameter -->
-    <xacro:property name="PI" value="3.1415926535897931"/>
+  <!-- Robot constants parameter -->
+  <!-- Y up,X front -->
+  <!-- Link 1 -->
+  <xacro:property name="mass1" value="0.710"/>
+  <xacro:property name="length1" value="0.05"/>
+  <xacro:property name="width1" value="0.05"/>
+  <xacro:property name="height1" value="${0.323+0.015}"/> <!-- length + joint -->
+  <xacro:property name="comx1" value="0.0"/>
+  <xacro:property name="comy1" value="0.0"/>
+  <xacro:property name="comz1" value="0.232"/>
+  <!-- Link 2 -->
+  <xacro:property name="mass2" value="0.351"/>
+  <xacro:property name="length2" value="0.05"/>
+  <xacro:property name="width2" value="0.05"/>
+  <xacro:property name="height2" value="0.265"/>
+  <xacro:property name="comx2" value="0.0"/>
+  <xacro:property name="comy2" value="0.0"/>
+  <xacro:property name="comz2" value="0.265"/>
+  <!-- World constants parameter -->
+  <xacro:property name="PI" value="3.1415926535897931"/>
 </robot>

Commit message: refine code & added joint_state_sub

File: visualizer/simulate_robot/urdf/acrobat_robot_IB.xacro (robot description, xacro)
@@ -1,57 +1,57 @@
 <?xml version="1.0"?>
 <robot name="IB_robot" xmlns:xacro="http://www.ros.org/wiki/xacro">
-    <!-- importing macro,constants,.gazebo files -->
-    <!-- robot mechanical parameters -->
-    <xacro:include filename="$(find simulate_robot)/urdf/system_constants.xacro"/>
-    <xacro:include filename="$(find simulate_robot)/urdf/link_macro.xacro"/>
-    <!-- Rviz material colors -->
-    <xacro:include filename="$(find simulate_robot)/urdf/material_parameter.xacro"/>
-    <!-- Gazebo custom tags,materials -->
-    <xacro:include filename="$(find simulate_robot)/urdf/acrobat_robot_IB.gazebo"/>
-    <!-- fixed base_link -->
-    <link name="world"/>
-    <joint name="world_fixed" type="fixed">
-        <parent link="world"/>
-        <child link="base"/>
-    </joint>
-    <!-- base_link -->
-    <link name="base">
-        <visual><!-- visual config -->
-            <origin xyz="0 0 ${(height1+height2+0.10)/2}" rpy="0 0 0"/>
-            <material name="white"/>
-            <geometry>
-                <box size="0.05 0.05 ${height1+height2+0.10}"/>
-            </geometry>
-        </visual>
-        <collision><!-- Gazebo collision config -->
-            <origin xyz="0 0 ${(height1+height2+10)/2}" rpy="0 0 0"/>
-            <geometry>
-                <box size="0.05 0.05 ${height1+height2+0.10}"/>
-            </geometry>
-        </collision>
-        <inertial>
-            <origin xyz="0 0 ${(height1+height2+10)/2}" rpy="0 0 0"/>
-            <mass value="100"/>
-            <inertia
-                ixx="10" ixy="0" ixz="0"
-                iyy="10" iyz="0"
-                izz="10"/>
-        </inertial>
-    </link>
-    <!-- 1st_link -->
-    <xacro:link_macro
-        suffix="1st_link" parent="base" type="continuous" color="orange"
-        width="${width1}" length="${length1}" height="${height1}" x_offset="0" y_offset="${width1}" z_offset="${height1+height2+0.10}"
-        mass="${mass1}" comx="${comx1}" comy="${comy1}" comz="${comz1}"
-        ixx="0.01" ixy="0" ixz="0"
-        iyy="0.01" iyz="0"
-        izz="0.0058"/>
-    <!-- 2nd_link -->
-    <xacro:link_macro
-        suffix="2nd_link" parent="1st_link" type="revolute" color="green"
-        width="${width2}" length="${length2}" height="${height2}" x_offset="0" y_offset="${width2}" z_offset="${height1}"
-        mass="${mass1}" comx="${comx2}" comy="${comy2}" comz="${comz2}"
-        ixx="0.01" ixy="0" ixz="0"
-        iyy="0.01" iyz="0"
-        izz="0.070"/>
+  <!-- importing macro,constants,.gazebo files -->
+  <!-- robot mechanical parameters -->
+  <xacro:include filename="$(find simulate_robot)/urdf/system_constants.xacro"/>
+  <xacro:include filename="$(find simulate_robot)/urdf/link_macro.xacro"/>
+  <!-- Rviz material colors -->
+  <xacro:include filename="$(find simulate_robot)/urdf/material_parameter.xacro"/>
+  <!-- Gazebo custom tags,materials -->
+  <xacro:include filename="$(find simulate_robot)/urdf/acrobat_robot_IB.gazebo"/>
+  <!-- fixed base_link -->
+  <link name="world"/>
+  <joint name="world_fixed" type="fixed">
+    <parent link="world"/>
+    <child link="base"/>
+  </joint>
+  <!-- base_link -->
+  <link name="base">
+    <visual><!-- visual config -->
+      <origin xyz="0 0 ${(height1+height2+0.10)/2}" rpy="0 0 0"/>
+      <material name="white"/>
+      <geometry>
+        <box size="0.05 0.05 ${height1+height2+0.10}"/>
+      </geometry>
+    </visual>
+    <collision><!-- Gazebo collision config -->
+      <origin xyz="0 0 ${(height1+height2+10)/2}" rpy="0 0 0"/>
+      <geometry>
+        <box size="0.05 0.05 ${height1+height2+0.10}"/>
+      </geometry>
+    </collision>
+    <inertial>
+      <origin xyz="0 0 ${(height1+height2+10)/2}" rpy="0 0 0"/>
+      <mass value="100"/>
+      <inertia
+        ixx="10" ixy="0" ixz="0"
+        iyy="10" iyz="0"
+        izz="10"/>
+    </inertial>
+  </link>
+  <!-- 1st_link -->
+  <xacro:link_macro
+    suffix="1st_link" parent="base" type="continuous" color="orange"
+    width="${width1}" length="${length1}" height="${height1}" x_offset="0" y_offset="${width1}" z_offset="${height1+height2+0.10}"
+    mass="${mass1}" comx="${comx1}" comy="${comy1}" comz="${comz1}"
+    ixx="0.01" ixy="0" ixz="0"
+    iyy="0.01" iyz="0"
+    izz="0.0058"/>
+  <!-- 2nd_link -->
+  <xacro:link_macro
+    suffix="2nd_link" parent="1st_link" type="revolute" color="green"
+    width="${width2}" length="${length2}" height="${height2}" x_offset="0" y_offset="${width2}" z_offset="${height1}"
+    mass="${mass1}" comx="${comx2}" comy="${comy2}" comz="${comz2}"
+    ixx="0.01" ixy="0" ixz="0"
+    iyy="0.01" iyz="0"
+    izz="0.070"/>
 </robot>

Commit message: edit model coordinate

File: visualizer/simulate_robot/urdf/acrobat_robot_IB.xacro (robot description, xacro)
@@ -39,8 +39,38 @@
     </inertial>
   </link>
+  <joint name="bar_conn" type="fixed">
+    <parent link="base"/>
+    <child link="bar"/>
+  </joint>
+  <!-- bar -->
+  <link name="bar">
+    <visual>
+      <origin xyz="0.0 ${0.1/2} ${(height1+height2+0.10)}" rpy="${PI/2} 0.0 0.0"/>
+      <material name="white"/>
+      <geometry>
+        <cylinder radius="0.01" length="0.10"/>
+      </geometry>
+    </visual>
+    <collision>
+      <origin xyz="0.0 ${0.1/2} ${(height1+height2+0.10)}" rpy="${PI/2} 0.0 0.0"/>
+      <material name="white"/>
+      <geometry>
+        <cylinder radius="0.01" length="0.10"/>
+      </geometry>
+    </collision>
+    <inertial>
+      <mass value="100"/>
+      <inertia
+        ixx="10" ixy="0" ixz="0"
+        iyy="10" iyz="0"
+        izz="10"/>
+        <origin xyz="0.0 ${0.1/2} ${(height1+height2+0.10)}" rpy="${PI/2} 0.0 0.0"/>
+    </inertial>
+  </link>
   <!-- 1st_link -->
   <xacro:link_macro
-    suffix="1st_link" parent="base" type="continuous" color="orange"
-    width="${width1}" length="${length1}" height="${height1}" x_offset="0" y_offset="${width1}" z_offset="${height1+height2+0.10}"
+    suffix="1st_link" parent="bar" type="continuous" color="orange"
+    width="${width1}" length="${length1}" height="${height1}"
+    x_offset="0" y_offset="${width1+0.1/2}" z_offset="${height1+height2+0.10}"
     mass="${mass1}" comx="${comx1}" comy="${comy1}" comz="${comz1}"
     ixx="0.01" ixy="0" ixz="0"
@@ -50,5 +80,6 @@
   <xacro:link_macro
     suffix="2nd_link" parent="1st_link" type="revolute" color="green"
-    width="${width2}" length="${length2}" height="${height2}" x_offset="0" y_offset="${width2}" z_offset="${height1}"
+    width="${width2}" length="${length2}" height="${height2}"
+    x_offset="0" y_offset="${width2}" z_offset="${height1}"
     mass="${mass1}" comx="${comx2}" comy="${comy2}" comz="${comz2}"
     ixx="0.01" ixy="0" ixz="0"

File: visualizer/simulate_robot/urdf/link_macro.xacro (robot description, xacro)
@@ -24,5 +24,5 @@
           <parent link="${parent}"/>
           <child link="${suffix}"/>
-          <origin xyz="${x_offset} ${y_offset} ${z_offset}" rpy="0 0 0"/>
+          <origin xyz="${x_offset} ${y_offset} ${z_offset}" rpy="${PI} 0 0"/>
           <limit effort="0" velocity="100"/>
           <axis xyz="0 1 0"/>
