Commit message: reshaped code

File: visualizer/simulate_robot/urdf/link_macro.xacro (robot description, xacro)
@@ -15,6 +15,6 @@
         <origin xyz="${x_offset} ${y_offset} ${z_offset}" rpy="0 0 0"/>
         <limit upper="${PI/2}" lower="${-PI/2}" effort="100" velocity="100"/>
-          <axis xyz="0 1 0"/>
-          <dynamics damping="0.1"/>
+        <axis xyz="0 1 0"/>
+        <dynamics damping="0.1"/>
       </joint>
     </xacro:if>

Commit message: edit controller launch

File: visualizer/simulate_robot/urdf/link_macro.xacro (robot description, xacro)
@@ -25,5 +25,5 @@
           <child link="${suffix}"/>
           <origin xyz="${x_offset} ${y_offset} ${z_offset}" rpy="${PI} 0 0"/>
-          <limit effort="0" velocity="100"/>
+          <limit effort="10" velocity="100"/>
           <axis xyz="0 1 0"/>
           <dynamics damping="0.00001"/>
